File: kicad/atomic_clock.kicad_sch (KiCad schematic)
At the start: 77 parts, among them J1 Conn_02x05_Top_Bottom, J10 Conn_02x05_Top_Bottom, J11 Conn_02x05_Top_Bottom, J12 USB_B_Micro, J13 Conn_ARM_JTAG_SWD_10, J14 Conn_01x03_Female, J2 Conn_02x05_Top_Bottom, J3 Conn_02x05_Top_Bottom, J4 Conn_02x05_Top_Bottom, J5 USB_B_Micro, J6 Conn_02x05_Top_Bottom, J7 Conn_02x05_Top_Bottom, J8 Conn_02x05_Top_Bottom, J9 Conn_02x05_Top_Bottom, Q1 Q_Dual_PMOS, SW1 SW_Push, U1 D198K, U10 ATSAMDA1E16B-A, U11 D198K, U12 D198K, U13 D198K, U14 D198K, U15 D198K, U16 MAX7221xWG, U17 D198K, U18 D198K, U19 D198K, U2 D198K, U20 NCP1117LPST33T3G, U21 mems_osc_st1630, U22 DHT20, U23 DCF77, U24 MCP73831-2-OT, U3 D198K, U4 D198K, U5 MAX7221xWG, U6 D198K, U7 D198K, U8 D198K, U9 D198K

Commit message: Start routing
Parts:
- D9: value D -> (none); footprint Diode_SMD:D_SMA -> (none)
- Q2: value (none) -> Q_Dual_PMOS; footprint (none) -> Package_TO_SOT_SMD:SOT-363_SC-70-6
- R10, R11, R12, R13, R14, R15, R7, R8: footprint (none) -> Resistor_SMD:R_0805_2012Metric
- U25: value (none) -> TXB0101
Connections:
- net 3DP2: no longer U19.5 (DP)
- net USB_PWR: now reaches D5.1 (K), D6.1 (K), D8.2 (A), Q2.1 (S), R10.1, U25.6 (VCCB)
- net 3IND: now reaches J11.7 (Pin_7)
- net 3IND: now also U19.5 (DP)
- net 1IND: now reaches J10.7 (Pin_7)
- net 1IND: now also U10.15 (PA14_SER2_PAD2/SER4_PAD2)
- no-connect marks 38 -> 35
Changed lines of the file:
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@@
   (no_connect (at 426.085 246.38))
   (no_connect (at 426.085 243.84))
-  (no_connect (at 426.085 238.76))
   (no_connect (at 58.42 135.255))
   (no_connect (at 84.455 135.255))
@@
   (no_connect (at 119.38 275.59))
   (no_connect (at 119.38 278.13))
-  (no_connect (at 309.245 121.285))
   (no_connect (at 119.38 243.84))
   (no_connect (at 301.625 121.285))
@@
   (no_connect (at 426.085 275.59))
   (no_connect (at 426.085 278.13))
-  (no_connect (at 426.085 270.51))
   (bus_entry (at 100.965 270.51) (size 2.54 2.54)
     (stroke (width 0) (type default) (color 0 0 0 0))
@@
     (stroke (width 0) (type default) (color 0 0 0 0))
   )
+  (wire (pts (xy 309.245 121.285) (xy 309.245 129.54))
+    (stroke (width 0) (type default) (color 0 0 0 0))
+  )
   (wire (pts (xy 481.965 297.18) (xy 485.14 297.18))
     (stroke (width 0) (type default) (color 0 0 0 0))
@@
     (stroke (width 0) (type default) (color 0 0 0 0))
   )
+  (wire (pts (xy 426.085 238.76) (xy 426.72 238.76))
+    (stroke (width 0) (type default) (color 0 0 0 0))
+  )
   (wire (pts (xy 147.32 184.15) (xy 147.32 187.96))
     (stroke (width 0) (type default) (color 0 0 0 0))
@@
     (stroke (width 0) (type default) (color 0 0 0 0))
   )
+  (wire (pts (xy 426.085 270.51) (xy 426.72 270.51))
+    (stroke (width 0) (type default) (color 0 0 0 0))
+  )
   (bus (pts (xy 404.495 297.18) (xy 404.495 299.72))
     (stroke (width 0) (type default) (color 0 0 0 0))
@@
     (effects (font (size 1.27 1.27)) (justify left bottom))
   )
+  (label "1IND" (at 426.72 238.76 0)
+    (effects (font (size 1.27 1.27)) (justify left bottom))
+  )
   (label "2s8" (at 300.355 318.77 0)
     (effects (font (size 1.27 1.27)) (justify left bottom))
   )
+  (label "1IND" (at 309.245 129.54 90)
+    (effects (font (size 1.27 1.27)) (justify left bottom))
+  )
   (label "2B1" (at 178.435 299.72 0)
     (effects (font (size 1.27 1.27)) (justify left bottom))
@@
     (effects (font (size 1.27 1.27)) (justify right bottom))
   )
-  (label "3DP2" (at 507.365 314.96 0)
+  (label "3IND" (at 507.365 314.96 0)
     (effects (font (size 1.27 1.27)) (justify left bottom))
   )
@@
     (effects (font (size 1.27 1.27)) (justify left bottom))
   )
+  (label "USB_PWR" (at 67.31 115.57 0)
+    (effects (font (size 1.27 1.27)) (justify left bottom))
+  )
   (label "1s12" (at 412.75 241.3 180)
     (effects (font (size 1.27 1.27)) (justify right bottom))
@@
     (effects (font (size 1.27 1.27)) (justify right bottom))
   )
+  (label "3IND" (at 426.72 270.51 0)
+    (effects (font (size 1.27 1.27)) (justify left bottom))
+  )
   (label "2E1" (at 254.635 307.34 0)
     (effects (font (size 1.27 1.27)) (justify left bottom))
@@
     (property "Reference" "R12" (id 0) (at 118.11 118.745 90))
     (property "Value" "10K" (id 1) (at 118.745 115.57 90))
-    (property "Footprint" "" (id 2) (at 118.745 117.348 90)
+    (property "Footprint" "Resistor_SMD:R_0805_2012Metric" (id 2) (at 118.745 117.348 90)
       (effects (font (size 1.27 1.27)) hide)
     )
@@
       (effects (font (size 1.27 1.27)) (justify left))
     )
-    (property "Value" "" (id 1) (at 102.362 86.1572 0)
+    (property "Value" "Q_Dual_PMOS" (id 1) (at 102.362 86.1572 0)
       (effects (font (size 1.27 1.27)) (justify left))
     )
-    (property "Footprint" "" (id 2) (at 98.425 84.455 0)
+    (property "Footprint" "Package_TO_SOT_SMD:SOT-363_SC-70-6" (id 2) (at 98.425 84.455 0)
       (effects (font (size 1.27 1.27)) hide)
     )
@@
     (property "Reference" "R7" (id 0) (at 49.53 50.5292 90))
     (property "Value" "10K" (id 1) (at 49.53 53.0661 90))
-    (property "Footprint" "" (id 2) (at 49.53 57.023 90)
+    (property "Footprint" "Resistor_SMD:R_0805_2012Metric" (id 2) (at 49.53 57.023 90)
       (effects (font (size 1.27 1.27)) hide)
     )
@@
     (in_bom yes) (on_board yes) (fields_autoplaced)
     (property "Reference" "U25" (id 0) (at 72.39 93.184 0))
-    (property "Value" "" (id 1) (at 72.39 90.6471 0))
+    (property "Value" "TXB0101" (id 1) (at 72.39 90.6471 0))
     (property "Footprint" "Package_TO_SOT_SMD:SOT-363_SC-70-6" (id 2) (at 46.99 71.755 0)
       (effects (font (size 1.27 1.27)) hide)
@@
     (property "Reference" "R14" (id 0) (at 41.91 50.5292 90))
     (property "Value" "10K" (id 1) (at 41.91 53.0661 90))
-    (property "Footprint" "" (id 2) (at 41.91 57.023 90)
+    (property "Footprint" "Resistor_SMD:R_0805_2012Metric" (id 2) (at 41.91 57.023 90)
       (effects (font (size 1.27 1.27)) hide)
     )
@@
     (property "Reference" "R10" (id 0) (at 102.87 118.745 90))
     (property "Value" "10K" (id 1) (at 103.505 115.57 90))
-    (property "Footprint" "" (id 2) (at 103.505 117.348 90)
+    (property "Footprint" "Resistor_SMD:R_0805_2012Metric" (id 2) (at 103.505 117.348 90)
       (effects (font (size 1.27 1.27)) hide)
     )
@@
     (property "Reference" "R15" (id 0) (at 49.53 41.6392 90))
     (property "Value" "10K" (id 1) (at 49.53 44.1761 90))
-    (property "Footprint" "" (id 2) (at 49.53 48.133 90)
+    (property "Footprint" "Resistor_SMD:R_0805_2012Metric" (id 2) (at 49.53 48.133 90)
       (effects (font (size 1.27 1.27)) hide)
     )
@@
     (property "Reference" "R13" (id 0) (at 41.91 41.6392 90))
     (property "Value" "10K" (id 1) (at 41.91 44.1761 90))
-    (property "Footprint" "" (id 2) (at 41.91 48.133 90)
+    (property "Footprint" "Resistor_SMD:R_0805_2012Metric" (id 2) (at 41.91 48.133 90)
       (effects (font (size 1.27 1.27)) hide)
     )
@@
       (effects (font (size 1.27 1.27)) (justify right))
     )
-    (property "Value" "D" (id 1) (at 117.602 96.3172 90)
+    (property "Value" "" (id 1) (at 117.602 96.3172 90)
       (effects (font (size 1.27 1.27)) (justify right))
     )
-    (property "Footprint" "Diode_SMD:D_SMA" (id 2) (at 115.57 94.615 0)
+    (property "Footprint" "" (id 2) (at 115.57 94.615 0)
       (effects (font (size 1.27 1.27)) hide)
     )
@@
     (property "Reference" "R8" (id 0) (at 102.235 52.07 90))
     (property "Value" "330R" (id 1) (at 102.87 55.245 90))
-    (property "Footprint" "" (id 2) (at 102.87 53.467 90)
+    (property "Footprint" "Resistor_SMD:R_0805_2012Metric" (id 2) (at 102.87 53.467 90)
       (effects (font (size 1.27 1.27)) hide)
     )
@@
     (property "Reference" "R11" (id 0) (at 110.49 118.745 90))
     (property "Value" "10K" (id 1) (at 111.125 115.57 90))
-    (property "Footprint" "" (id 2) (at 111.125 117.348 90)
+    (property "Footprint" "Resistor_SMD:R_0805_2012Metric" (id 2) (at 111.125 117.348 90)
       (effects (font (size 1.27 1.27)) hide)
     )

Commit message: Routed PCB
Parts:
- added R16: (no value), symbol Device:R
- D9: value (none) -> D; footprint (none) -> Diode_SMD:D_SMA
Connections:
- net 1IND: now also R16.2; no longer U10.15 (PA14_SER2_PAD2/SER4_PAD2)
- net NCP_IN: now reaches C2.1, D8.1 (K), D9.1 (K), U20.3 (VIN)
- net USB+ renamed USB_P
- net USB- renamed USB_N
- new net: R16.1, U10.15 (PA14_SER2_PAD2/SER4_PAD2)
Changed lines of the file:
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@@
   (no_connect (at 58.42 135.255))
   (no_connect (at 84.455 135.255))
+  (no_connect (at 321.945 121.285))
   (no_connect (at 220.98 246.38))
   (no_connect (at 375.285 275.59))
   (no_connect (at 344.805 121.285))
-  (no_connect (at 321.945 121.285))
   (no_connect (at 319.405 121.285))
   (no_connect (at 119.38 246.38))
@@
     (stroke (width 0) (type default) (color 0 0 0 0))
   )
-  (wire (pts (xy 316.865 132.08) (xy 299.085 132.08))
+  (wire (pts (xy 316.865 147.32) (xy 299.085 147.32))
     (stroke (width 0) (type default) (color 0 0 0 0))
   )
@@
     (stroke (width 0) (type default) (color 0 0 0 0))
   )
-  (wire (pts (xy 314.96 133.985) (xy 314.96 184.15))
+  (wire (pts (xy 314.96 149.86) (xy 314.96 184.15))
     (stroke (width 0) (type default) (color 0 0 0 0))
   )
@@
     (stroke (width 0) (type default) (color 0 0 0 0))
   )
-  (wire (pts (xy 296.545 121.285) (xy 296.545 133.985))
+  (wire (pts (xy 296.545 121.285) (xy 296.545 149.86))
     (stroke (width 0) (type default) (color 0 0 0 0))
   )
@@
     (stroke (width 0) (type default) (color 0 0 0 0))
   )
-  (wire (pts (xy 294.005 135.89) (xy 313.055 135.89))
+  (wire (pts (xy 294.005 152.4) (xy 313.055 152.4))
     (stroke (width 0) (type default) (color 0 0 0 0))
   )
@@
     (stroke (width 0) (type default) (color 0 0 0 0))
   )
-  (wire (pts (xy 316.865 182.245) (xy 316.865 132.08))
+  (wire (pts (xy 316.865 182.245) (xy 316.865 147.32))
     (stroke (width 0) (type default) (color 0 0 0 0))
   )
@@
     (stroke (width 0) (type default) (color 0 0 0 0))
   )
-  (wire (pts (xy 296.545 133.985) (xy 314.96 133.985))
+  (wire (pts (xy 296.545 149.86) (xy 314.96 149.86))
     (stroke (width 0) (type default) (color 0 0 0 0))
   )
@@
     (stroke (width 0) (type default) (color 0 0 0 0))
   )
-  (wire (pts (xy 294.005 121.285) (xy 294.005 135.89))
+  (wire (pts (xy 294.005 121.285) (xy 294.005 152.4))
     (stroke (width 0) (type default) (color 0 0 0 0))
   )
@@
     (stroke (width 0) (type default) (color 0 0 0 0))
   )
-  (wire (pts (xy 313.055 135.89) (xy 313.055 180.34))
+  (wire (pts (xy 313.055 152.4) (xy 313.055 180.34))
     (stroke (width 0) (type default) (color 0 0 0 0))
   )
@@
     (stroke (width 0) (type default) (color 0 0 0 0))
   )
-  (wire (pts (xy 299.085 132.08) (xy 299.085 121.285))
+  (wire (pts (xy 299.085 147.32) (xy 299.085 121.285))
     (stroke (width 0) (type default) (color 0 0 0 0))
   )
@@
     (effects (font (size 1.27 1.27)) (justify left bottom))
   )
+  (label "NCP_IN" (at 120.015 101.6 0)
+    (effects (font (size 1.27 1.27)) (justify left bottom))
+  )
   (label "2F1" (at 178.435 309.88 0)
     (effects (font (size 1.27 1.27)) (justify left bottom))
@@
     (effects (font (size 1.27 1.27)) (justify left bottom))
   )
+  (label "1IND" (at 309.245 137.16 270)
+    (effects (font (size 1.27 1.27)) (justify right bottom))
+  )
   (label "3D2" (at 432.435 304.8 0)
     (effects (font (size 1.27 1.27)) (justify left bottom))
@@
     (effects (font (size 1.27 1.27)) (justify left bottom))
   )
-  (label "1IND" (at 309.245 129.54 90)
-    (effects (font (size 1.27 1.27)) (justify left bottom))
-  )
   (label "2B1" (at 178.435 299.72 0)
     (effects (font (size 1.27 1.27)) (justify left bottom))
@@
     (effects (font (size 1.27 1.27)) (justify left bottom))
   )
-  (label "USB+" (at 337.185 131.445 90)
+  (label "USB_P" (at 337.185 131.445 90)
     (effects (font (size 1.27 1.27)) (justify left bottom))
   )
@@
     (effects (font (size 1.27 1.27)) (justify right bottom))
   )
-  (label "USB-" (at 334.645 131.445 90)
+  (label "USB_N" (at 334.645 131.445 90)
     (effects (font (size 1.27 1.27)) (justify left bottom))
   )
@@
     (effects (font (size 1.27 1.27)) (justify right bottom))
   )
-  (label "USB-" (at 90.17 132.715 0)
+  (label "USB_N" (at 90.17 132.715 0)
     (effects (font (size 1.27 1.27)) (justify left bottom))
   )
@@
     (effects (font (size 1.27 1.27)) (justify left bottom))
   )
-  (label "USB+" (at 90.17 130.175 0)
+  (label "USB_P" (at 90.17 130.175 0)
     (effects (font (size 1.27 1.27)) (justify left bottom))
   )
@@
     (pin "5")
   )
+  (symbol (lib_id "Device:R") (at 309.245 133.35 0) (unit 1)
+    (in_bom yes) (on_board yes)
+    (property "Reference" "R16" (id 0) (at 306.705 132.715 90))
+    (property "Value" "" (id 1) (at 311.4239 133.35 90))
+    (property "Footprint" "" (id 2) (at 307.467 133.35 90)
+      (effects (font (size 1.27 1.27)) hide)
+    )
+    (property "Datasheet" "~" (id 3) (at 309.245 133.35 0)
+      (effects (font (size 1.27 1.27)) hide)
+    )
+    (pin "1")
+    (pin "2")
+  )
   (symbol (lib_id "Device:R") (at 49.53 55.245 270) (mirror x) (unit 1)
     (in_bom yes) (on_board yes) (fields_autoplaced)
@@
       (effects (font (size 1.27 1.27)) (justify right))
     )
-    (property "Value" "" (id 1) (at 117.602 96.3172 90)
+    (property "Value" "D" (id 1) (at 117.602 96.3172 90)
       (effects (font (size 1.27 1.27)) (justify right))
     )
-    (property "Footprint" "" (id 2) (at 115.57 94.615 0)
+    (property "Footprint" "Diode_SMD:D_SMA" (id 2) (at 115.57 94.615 0)
       (effects (font (size 1.27 1.27)) hide)
     )
@@
       (reference "R15") (unit 1) (value "10K") (footprint "Resistor_SMD:R_0805_2012Metric")
     )
+    (path "/1de17caf-1a38-49fb-8dfa-f4155d8523b6"
+      (reference "R16") (unit 1) (value "220R") (footprint "Resistor_SMD:R_0805_2012Metric")
+    )
     (path "/944d7a4d-7ccb-431b-bb4e-a618ca75c13a"
