File: kicad/atomic_clock.kicad_sch (KiCad schematic)
At the start: 80 parts

Commit message: Fix short circuit in LDO symbol and footprint
The heatsink on the NCP1117LP LDO was incorrectly wired to GND, while
this pin is actually connected to Vout, causing a short circuit on
the assembled board.

https://twitter.com/erikvanzijst/status/1541097400571420672
Parts:
- BT1: value (none) -> Varta CP1654 A3; footprint (none) -> local_footprints:Battery_pads
- C1, C4, C6, C7, C8: value (none) -> 100nF 885012207016; footprint (none) -> Capacitor_SMD:C_0805_2012Metric
- C10, C9: value (none) -> 4.7uF CL21A475KPFNNNE; footprint (none) -> Capacitor_SMD:C_0805_2012Metric
- C11, C2, C3: value (none) -> 10uF CL21A106KPFNNNF; footprint (none) -> Capacitor_SMD:C_0805_2012Metric
- C5: value (none) -> 1uF 885012207051; footprint (none) -> Capacitor_SMD:C_0805_2012Metric
- D1, D2, D3, D4: value (none) -> LED LTL-1224A; footprint (none) -> local_footprints:LED_D2.0mm_W4.8mm_H2.5mm_FlatTop
- D10, D7: value (none) -> LED HSMS-C150; footprint (none) -> LED_SMD:LED_1206_3216Metric_Pad1.42x1.75mm_HandSolder
- D5, D6, D8, D9: value (none) -> Diode S1M-13-F; footprint (none) -> Diode_SMD:D_SMA
- J1, J10, J11, J2, J3, J4, J6, J7, J8, J9: value (none) -> Conn_02x05_Top_Bottom; footprint (none) -> Connector_PinHeader_2.54mm:PinHeader_2x05_P2.54mm_Vertical
- J12: value (none) -> USB_B_Micro 10118194-0001LF; footprint (none) -> Connector_USB:USB_Micro-B_Amphenol_10118194_Horizontal
- J13: value (none) -> ARM_JTAG_SWD_10 3220-10-0100-00; footprint (none) -> local_footprints:sam_swd_header
- J14: value (none) -> Conn_01x03_Female; footprint (none) -> Connector_PinSocket_2.54mm:PinSocket_1x03_P2.54mm_Vertical
- J5: value (none) -> USB_B_Micro 1051330001; footprint (none) -> Connector_USB:USB_Micro-B_Molex-105133-0001
- Q1, Q2: value (none) -> Q_Dual_PMOS; footprint (none) -> Package_TO_SOT_SMD:SOT-363_SC-70-6
- R1, R10, R11, R12, R13, R14, R15, R3, R4, R5, R7, R9: value (none) -> 10K; footprint (none) -> Resistor_SMD:R_0805_2012Metric
- R16: value (none) -> 220R; footprint (none) -> Resistor_SMD:R_0805_2012Metric
- R2: value (none) -> 1K; footprint (none) -> Resistor_SMD:R_0805_2012Metric
- R6: value (none) -> LDR NSL-19M51; footprint (none) -> OptoDevice:R_LDR_4.9x4.2mm_P2.54mm_Vertical
- R8: value (none) -> 470R; footprint (none) -> Resistor_SMD:R_0805_2012Metric
- SW1: value (none) -> SW_Push; footprint (none) -> Button_Switch_SMD:SW_SPST_TL3342
- U1, U11, U12, U13, U14, U15, U17, U18, U19, U2, U3, U4, U6, U7, U8, U9: value (none) -> D198K; footprint (none) -> Display_7Segment:D1X8K
- U10: value (none) -> ATSAMDA1E16B-A; footprint (none) -> Package_QFP:TQFP-32_7x7mm_P0.8mm
- U16, U5: value (none) -> MAX7221xWG; footprint (none) -> Package_SO:SOIC-24W_7.5x15.4mm_P1.27mm
- U20: value (none) -> NCP1117LPST33T3G; footprint (none) -> Package_TO_SOT_SMD:SOT-223
- U21: value (none) -> mems_osc_st1630; footprint (none) -> Package_TO_SOT_SMD:SOT-23-5
- U22: value (none) -> DHT20; footprint (none) -> local_footprints:DHT20
- U23: value (none) -> DCF77; footprint (none) -> local_footprints:DCF77 receiver module
- U24: value (none) -> MCP73831-2-OT; footprint (none) -> Package_TO_SOT_SMD:SOT-23-5
- U25: value (none) -> TXB0101; footprint (none) -> Package_TO_SOT_SMD:SOT-363_SC-70-6
Connections:
- net 3.3V: now also U20.4 (VOUT)
- net GND: no longer U20.4 (SINK)
